File: board/pbrick.sch (KiCad schematic (older format))
At the start: 31 parts, among them J1 JST_2MM_MALE, J2 QWIIC, J3 B4B-XH-A(LF)(SN), J4 B4B-XH-A(LF)(SN), J5 U.FL2PIN, P0 SWD, U1 ADP3330ARTZ-5-RL7, U2 MIC5219-3.3YML-TR, U3 TB6612FNG

Commit message: Merging board source code with firmware
Parts:
- removed C5: .22uF, Capacitors:0603, symbol pbrick-rescue:CAPACITOR_NP_0603-MF_Passives
- removed C7: 16V 10uF, EIA3528, symbol pbrick-rescue:68UF-POLAR-EIA3528-10V-10%_TANT_-SparkFun-Capacitors
- removed U3: TB6612FNG, Package_SO:SSOP-24_5.3x8.2mm_P0.65mm, symbol Driver_Motor:TB6612FNG
- added C14: 270pF 0603, Capacitors:0603, symbol pbrick-rescue:CAPACITOR_NP_0603-MF_Passives
- added C15: 100nF 0603, Capacitors:0603, symbol pbrick-rescue:CAPACITOR_NP_0603-MF_Passives
- added C16: 22UF 10% 25V, Capacitor_Tantalum_SMD:CP_EIA-6032-15_Kemet-U_Pad2.25x2.35mm_HandSolder, symbol Device:CP1
- added H1, H2: MountingHole_Pad, symbol Mechanical:MountingHole_Pad
- added R9: 5.1K, Resistors:0603, symbol pbrick-rescue:RESISTOR_0603-MF_Passives
- added U1: TB67H420FTG(O,EL), IC_TB67H420FTG(O,EL), symbol TB67H420FTG_O_EL_:TB67H420FTG(O,EL)
- renumbered C6 to C10, C26 to C11, C27 to C12, C28 to C13, C2 to C6, C8 to C7, C9 to C8, C21 to C9, J4 to J1, J3 to J2, J2 to J3, J1 to J4, P0 to P1, R7 to R6, U1 to U3
Connections:
- wire segments 90 -> 97
- no-connect marks 5 -> 7
Other:
- moved on the sheet: LED1, R1, R2, R3

Commit message: non-16mm
Parts:
- removed J1, J2: B4B-XH-A(LF)(SN), JST_B4B-XH-A(LF)(SN), symbol pbrick-rescue:B4B-XH-A(LF)(SN)-B4B-XH-A_LF__SN_
- added J1: S6B-PH-SM4-TB(LF)(SN), JST_S6B-PH-SM4-TB(LF)(SN), symbol S6B-PH-SM4-TB_LF__SN_:S6B-PH-SM4-TB(LF)(SN)
- C1: Description CAP CER 0.47UF 16V X5R 0603 -> CAP CER 0.47UF 25V X7R 0603; Digi-Key_PN 732-7912-1-ND -> 732-7993-1-ND; MPN 885012106015 -> 885012206075
- C12, C13, H1, H2, J3, J4, P1, S1: fit_field (none) -> dnp
- C14: Digi-Key_PN 732-7965-1-ND -> 732-7989-1-ND; MPN 885012206046 -> 885012206071
- C15: Description CAP CER 0.1UF 16V X7R 0603 -> CAP CER 0.1UF 25V X7R 0603; Digi-Key_PN 732-7965-1-ND -> 732-7989-1-ND; MPN 885012206046 -> 885012206071
- C16: Digi-Key_PN (none) -> 718-1511-1-ND; DigiKey_PN 718-1511-1-ND -> (none)
- C4: value 2.2uf -> 2.2uF
- C6: Digi-Key_PN 732-7912-1-ND -> 732-7993-1-ND; MPN 885012106015 -> 885012206075
- R9: Digi-Key_PN RHM10KDCT-ND -> (none); DigiKey_PN (none) -> RHM10KDCT-ND
Connections:
- no-connect marks 7 -> 8
Changed lines of the file:
@@
 F 5 "C&K SWITCHES" H 5650 1400 50  0001 L BNN "Field5"
 F 6 "Manufacturer Recommendations" H 5650 1400 50  0001 L BNN "Field6"
+F 7 "dnp" H 5650 1400 50  0001 C CNN "fit_field"
 	1    5650 1400
 	1    0    0    -1
@@
 F 2 "Connectors:SAMTECH_FTSH-105-01" H 5800 5100 50  0001 C CNN
 F 3 "http://infocenter.arm.com/help/topic/com.arm.doc.ddi0314h/DDI0314H_coresight_components_trm.pdf" V 5450 3850 50  0001 C CNN
+F 4 "dnp" V 5800 5100 50  0001 C CNN "fit_field"
 	1    5800 5100
 	0    1    1    0
@@
 F 2 "Capacitors:0603" H 3800 1810 20  0001 C CNN
 F 3 "https://www.we-online.de/katalog/datasheet/885012106015.pdf" H 3550 1900 60  0001 C CNN
-F 4 "732-7912-1-ND" H 3550 1900 50  0001 C CNN "Digi-Key_PN"
+F 4 "732-7993-1-ND" H 3550 1900 50  0001 C CNN "Digi-Key_PN"
 F 5 "Würth Elektronik" H 3550 1900 50  0001 C CNN "Manufacturer"
-F 6 "885012106015" H 3550 1900 50  0001 C CNN "MPN"
+F 6 "885012206075" H 3550 1900 50  0001 C CNN "MPN"
 F 7 "CAP CER 0.47UF 16V X5R 0603" H 3550 1900 50  0001 C CNN "Description"
 	1    3550 1900
@@
 	1650 1500 1900 1500
 Connection ~ 1650 1500
-$Comp
-L pbrick-rescue:CAPACITOR_NP_0603-MF_Passives C1
-U 1 1 5F17448E
-P 1650 1600
-F 0 "C1" H 1450 1650 45  0000 L CNN
-F 1 "470nF 0603" H 1150 1550 45  0000 L CNN
-F 2 "Capacitors:0603" H 1900 1510 20  0001 C CNN
-F 3 "https://www.we-online.de/katalog/datasheet/885012106015.pdf" H 1650 1600 60  0001 C CNN
-F 4 "732-7912-1-ND" H 1650 1600 50  0001 C CNN "Digi-Key_PN"
-F 5 "Würth Elektronik" H 1650 1600 50  0001 C CNN "Manufacturer"
-F 6 "885012106015" H 1650 1600 50  0001 C CNN "MPN"
-F 7 "CAP CER 0.47UF 16V X5R 0603" H 1650 1600 50  0001 C CNN "Description"
-	1    1650 1600
-	1    0    0    -1
-$EndComp
 Wire Wire Line
 	1900 1900 2050 1900
@@
 P 3150 3750
 F 0 "C4" H 3248 3792 45  0000 L CNN
-F 1 "2.2uf" H 3248 3708 45  0000 L CNN
+F 1 "2.2uF" H 3248 3708 45  0000 L CNN
 F 2 "Capacitors:0603" H 3400 3660 20  0001 C CNN
 F 3 "https://katalog.we-online.de/pbs/datasheet/885012106018.pdf" H 3150 3750 60  0001 C CNN
@@
 P0.00
 $Comp
-L power:Earth #PWR016
-U 1 1 5F18A29B
-P 4500 7450
-F 0 "#PWR016" H 4500 7200 50  0001 C CNN
-F 1 "Earth" H 4500 7300 50  0001 C CNN
-F 2 "" H 4500 7450 50  0001 C CNN
-F 3 "~" H 4500 7450 50  0001 C CNN
-	1    4500 7450
-	1    0    0    -1
-$EndComp
-Text Label 4500 7350 0    50   ~ 0
-M0_0
-Text Label 4500 7250 0    50   ~ 0
-M0_1
-$Comp
 L pbrick-rescue:CAPACITOR_NP_0603-MF_Passives C12
 U 1 1 5F1FECBD
@@
 F 6 "885012006019" H 9250 1200 50  0001 C CNN "MPN"
 F 7 "CAP CER 22PF 16V C0G/NP0 0603" H 9250 1200 50  0001 C CNN "Description"
+F 8 "dnp" H 9250 1200 50  0001 C CNN "fit_field"
 	1    9250 1200
 	1    0    0    -1
@@
 F 6 "885012006019" H 9250 1550 50  0001 C CNN "MPN"
 F 7 "CAP CER 22PF 16V C0G/NP0 0603" H 9250 1550 50  0001 C CNN "Description"
+F 8 "dnp" H 9250 1550 50  0001 C CNN "fit_field"
 	1    9250 1550
 	1    0    0    -1
@@
 	2200 3550 2200 3650
 $Comp
-L power:VDD #PWR013
-U 1 1 5F919418
-P 3800 7150
-F 0 "#PWR013" H 3800 7000 50  0001 C CNN
-F 1 "VDD" H 3815 7323 50  0000 C CNN
-F 2 "" H 3800 7150 50  0001 C CNN
-F 3 "" H 3800 7150 50  0001 C CNN
-	1    3800 7150
-	1    0    0    -1
-$EndComp
-$Comp
-L power:Earth #PWR014
-U 1 1 5F919422
-P 3800 7450
-F 0 "#PWR014" H 3800 7200 50  0001 C CNN
-F 1 "Earth" H 3800 7300 50  0001 C CNN
-F 2 "" H 3800 7450 50  0001 C CNN
-F 3 "~" H 3800 7450 50  0001 C CNN
-	1    3800 7450
-	1    0    0    -1
-$EndComp
-Text Label 3800 7350 0    50   ~ 0
-M1_0
-Text Label 3800 7250 0    50   ~ 0
-M1_1
-$Comp
 L pbrick-rescue:U.FL2PIN-SparkFun-Connectors J5
 U 1 1 5F205E4A
@@
 $EndComp
 $Comp
-L power:VDD #PWR015
-U 1 1 5F189B11
-P 4500 7150
-F 0 "#PWR015" H 4500 7000 50  0001 C CNN
-F 1 "VDD" H 4515 7323 50  0000 C CNN
-F 2 "" H 4500 7150 50  0001 C CNN
-F 3 "" H 4500 7150 50  0001 C CNN
-	1    4500 7150
-	1    0    0    -1
-$EndComp
-$Comp
 L pbrick-rescue:I2C_STANDARDQWIIC-SparkFun-Connectors J3
 U 1 1 5F11DB2A
@@
 F 3 "" H 5500 7300 50  0001 C CNN
 F 4 "CONN-13729" H 5458 7731 60  0001 C CNN "Field4"
+F 5 "dnp" V 5500 7300 50  0001 C CNN "fit_field"
 	1    5500 7300
 	0    -1   -1   0
@@
 F 2 "" H 7100 5800 50  0001 C CNN
 F 3 "~" H 7100 5800 50  0001 C CNN
+F 4 "dnp" H 7100 5800 50  0001 C CNN "fit_field"
 	1    7100 5800
 	-1   0    0    1
@@
 F 2 "" H 7100 6250 50  0001 C CNN
 F 3 "~" H 7100 6250 50  0001 C CNN
+F 4 "dnp" H 7100 6250 50  0001 C CNN "fit_field"
 	1    7100 6250
 	-1   0    0    1
@@
 F 2 "Resistors:0603" H 3700 5910 20  0001 C CNN
 F 3 "https://d1d2qsbl8m0m72.cloudfront.net/en/products/databook/datasheet/passive/resistor/chip_resistor/esr-e.pdf" H 3450 6000 60  0001 C CNN
-F 4 "RHM10KDCT-ND" H 3450 6000 50  0001 C CNN "Digi-Key_PN"
+F 4 "RHM10KDCT-ND" H 3450 6000 50  0001 C CNN "DigiKey_PN"
 F 5 "Rohm Semiconductor" H 3450 6000 50  0001 C CNN "Manufacturer"
 F 6 "ESR03EZPJ103" H 3450 6000 50  0001 C CNN "MPN"
@@
 F 2 "Capacitors:0603" H 3500 5810 20  0001 C CNN
 F 3 "https://www.we-online.de/katalog/datasheet/885012106015.pdf" H 3250 5900 60  0001 C CNN
-F 4 "732-7965-1-ND" V 3250 5900 50  0001 C CNN "Digi-Key_PN"
+F 4 "732-7989-1-ND" V 3250 5900 50  0001 C CNN "Digi-Key_PN"
 F 5 "Würth Elektronik" V 3250 5900 50  0001 C CNN "Manufacturer"
-F 6 "885012206046" V 3250 5900 50  0001 C CNN "MPN"
+F 6 "885012206071" V 3250 5900 50  0001 C CNN "MPN"
 F 7 "CAP CER 0.1UF 16V X7R 0603" V 3250 5900 50  0001 C CNN "Description"
 	1    3250 5900
@@
 F 2 "Capacitors:0603" H 3700 5210 20  0001 C CNN
 F 3 "https://www.we-online.de/katalog/datasheet/885012106015.pdf" H 3450 5300 60  0001 C CNN
-F 4 "732-7965-1-ND" V 3450 5300 50  0001 C CNN "Digi-Key_PN"
+F 4 "732-7989-1-ND" V 3450 5300 50  0001 C CNN "Digi-Key_PN"
 F 5 "Würth Elektronik" V 3450 5300 50  0001 C CNN "Manufacturer"
-F 6 "885012206046" V 3450 5300 50  0001 C CNN "MPN"
-F 7 "CAP CER 0.1UF 16V X7R 0603" V 3450 5300 50  0001 C CNN "Description"
+F 6 "885012206071" V 3450 5300 50  0001 C CNN "MPN"
+F 7 "CAP CER 0.1UF 25V X7R 0603" V 3450 5300 50  0001 C CNN "Description"
 	1    3450 5300
 	1    0    0    -1
@@
 F 4 "Vishay Sprague" H 3650 5250 50  0001 C CNN "Manufacturer"
 F 5 "TR3C226K025C0400" H 3650 5250 50  0001 C CNN "MPN"
-F 6 "718-1511-1-ND" H 3650 5250 50  0001 C CNN "DigiKey_PN"
+F 6 "718-1511-1-ND" H 3650 5250 50  0001 C CNN "Digi-Key_PN"
 F 7 "CAP TANT 22UF 10% 25V 2312" H 3650 5250 50  0001 C CNN "Description"
 	1    3650 5250
@@
 NoConn ~ 2750 6200
 NoConn ~ 2750 6300
-$Comp
-L pbrick-rescue:B4B-XH-A(LF)(SN)-B4B-XH-A_LF__SN_ J2
-U 1 1 5F166103
-P 4200 7350
-F 0 "J2" H 4307 7817 50  0000 C CNN
-F 1 "B4B-XH-A(LF)(SN)" H 4300 7000 50  0001 C CNN
-F 2 "JST_B4B-XH-A(LF)(SN)" H 4200 7350 50  0001 L BNN
-F 3 "NA" H 4200 7350 50  0001 L BNN
-F 4 "Manufacturer Recommendation" H 4200 7350 50  0001 L BNN "Field4"
-F 5 "JST Sales America Inc" H 4200 7350 50  0001 L BNN "Field5"
-	1    4200 7350
-	1    0    0    -1
-$EndComp
-$Comp
-L pbrick-rescue:B4B-XH-A(LF)(SN)-B4B-XH-A_LF__SN_ J1
-U 1 1 5F91940E
-P 3500 7350
-F 0 "J1" H 3607 7817 50  0000 C CNN
-F 1 "B4B-XH-A(LF)(SN)" H 3600 7000 50  0001 C CNN
-F 2 "JST_B4B-XH-A(LF)(SN)" H 3500 7350 50  0001 L BNN
-F 3 "NA" H 3500 7350 50  0001 L BNN
-F 4 "Manufacturer Recommendation" H 3500 7350 50  0001 L BNN "Field4"
-F 5 "JST Sales America Inc" H 3500 7350 50  0001 L BNN "Field5"
-	1    3500 7350
-	1    0    0    -1
-$EndComp
 $Comp
 L pbrick-rescue:JST_2MM_MALE-SparkFun-Connectors J4
@@
 F 3 "" H 6400 7300 50  0001 C CNN
 F 4 "CONN-11443" V 6650 7100 60  0001 L CNN "Field4"
+F 5 "dnp" H 6400 7300 50  0001 C CNN "fit_field"
 	1    6400 7300
 	-1   0    0    1
@@
 	-1   0    0    1
 $EndComp
+$Comp
+L pbrick-rescue:CAPACITOR_NP_0603-MF_Passives C1
+U 1 1 5F17448E
+P 1650 1600
+F 0 "C1" H 1450 1650 45  0000 L CNN
+F 1 "470nF 0603" H 1150 1550 45  0000 L CNN
+F 2 "Capacitors:0603" H 1900 1510 20  0001 C CNN
+F 3 "https://www.we-online.de/katalog/datasheet/885012106015.pdf" H 1650 1600 60  0001 C CNN
+F 4 "732-7993-1-ND" H 1650 1600 50  0001 C CNN "Digi-Key_PN"
+F 5 "Würth Elektronik" H 1650 1600 50  0001 C CNN "Manufacturer"
+F 6 "885012206075" H 1650 1600 50  0001 C CNN "MPN"
+F 7 "CAP CER 0.47UF 25V X7R 0603" H 1650 1600 50  0001 C CNN "Description"
+	1    1650 1600
+	1    0    0    -1
+$EndComp
+NoConn ~ 3650 7000
+Text Label 4250 7000 1    50   ~ 0
+M0_0
+Text Label 4150 7000 1    50   ~ 0
+M0_1
+Text Label 4050 7000 1    50   ~ 0
+M1_0
+Text Label 3950 7000 1    50   ~ 0
+M1_1
+$Comp
+L power:Earth #PWR0109
+U 1 1 5FF3EB22
+P 3850 7000
+F 0 "#PWR0109" H 3850 6750 50  0001 C CNN
+F 1 "Earth" H 3850 6850 50  0001 C CNN
+F 2 "" H 3850 7000 50  0001 C CNN
+F 3 "~" H 3850 7000 50  0001 C CNN
+	1    3850 7000
+	-1   0    0    1
+$EndComp
+$Comp
+L power:VDD #PWR013
+U 1 1 5F919418
+P 4350 7000
+F 0 "#PWR013" H 4350 6850 50  0001 C CNN
+F 1 "VDD" H 4365 7173 50  0000 C CNN
+F 2 "" H 4350 7000 50  0001 C CNN
+F 3 "" H 4350 7000 50  0001 C CNN
+	1    4350 7000
+	1    0    0    -1
+$EndComp
+$Comp
+L S6B-PH-SM4-TB_LF__SN_:S6B-PH-SM4-TB(LF)(SN) J1
+U 1 1 5FF58FC9
+P 4050 7300
+F 0 "J1" V 4450 7250 50  0000 L CNN
+F 1 "S6B-PH-SM4-TB(LF)(SN)" V 4350 6800 50  0000 L CNN
+F 2 "JST_S6B-PH-SM4-TB(LF)(SN)" H 4050 7300 50  0001 L BNN
+F 3 "" H 4050 7300 50  0001 L BNN
+F 4 "Manufacturer Recommendation" H 4050 7300 50  0001 L BNN "STANDARD"
+F 5 "JST" H 4050 7300 50  0001 L BNN "MANUFACTURER"
+	1    4050 7300
+	0    1    1    0
+$EndComp
 $EndSCHEMATC

Commit message: Converting to 24mm x 45mm board
Parts:
- removed J1: S6B-PH-SM4-TB(LF)(SN), JST_S6B-PH-SM4-TB(LF)(SN), symbol S6B-PH-SM4-TB_LF__SN_:S6B-PH-SM4-TB(LF)(SN)
- removed J4: JST_2MM_MALE, JST-2-SMD, symbol pbrick-rescue:JST_2MM_MALE-SparkFun-Connectors
- added J1: S8B-PH-SM4-TB_LF__SN_, S8BPHSM4TBLFSN, symbol S8B-PH-SM4-TB_LF__SN_:S8B-PH-SM4-TB_LF__SN_
Connections:
- no-connect marks 8 -> 9
Changed lines of the file:
@@
 NoConn ~ 2750 6300
-$Comp
-L pbrick-rescue:JST_2MM_MALE-SparkFun-Connectors J4
-U 1 1 5F132F9C
-P 6400 7300
-F 0 "J4" H 6350 7600 45  0000 L CNN
-F 1 "JST_2MM_MALE" H 6500 7100 45  0001 L BNN
-F 2 "JST-2-SMD" H 6400 7650 20  0001 C CNN
-F 3 "" H 6400 7300 50  0001 C CNN
-F 4 "CONN-11443" V 6650 7100 60  0001 L CNN "Field4"
-F 5 "dnp" H 6400 7300 50  0001 C CNN "fit_field"
-	1    6400 7300
-	-1   0    0    1
-$EndComp
-$Comp
-L power:VDD #PWR023
-U 1 1 5F16990D
-P 6350 7100
-F 0 "#PWR023" H 6350 6950 50  0001 C CNN
-F 1 "VDD" H 6365 7273 50  0000 C CNN
-F 2 "" H 6350 7100 50  0001 C CNN
-F 3 "" H 6350 7100 50  0001 C CNN
-	1    6350 7100
-	1    0    0    -1
-$EndComp
-$Comp
-L power:Earth #PWR025
-U 1 1 5F134828
-P 6450 7100
-F 0 "#PWR025" H 6450 6850 50  0001 C CNN
-F 1 "Earth" H 6450 6950 50  0001 C CNN
-F 2 "" H 6450 7100 50  0001 C CNN
-F 3 "~" H 6450 7100 50  0001 C CNN
-	1    6450 7100
-	-1   0    0    1
-$EndComp
 $Comp
 L pbrick-rescue:CAPACITOR_NP_0603-MF_Passives C1
@@
 	1    0    0    -1
 $EndComp
-NoConn ~ 3650 7000
+NoConn ~ 4250 7900
+Text Label 4150 7000 1    50   ~ 0
+M0_0
 Text Label 4250 7000 1    50   ~ 0
-M0_0
-Text Label 4150 7000 1    50   ~ 0
 M0_1
-Text Label 4050 7000 1    50   ~ 0
+Text Label 3850 7000 1    50   ~ 0
 M1_0
-Text Label 3950 7000 1    50   ~ 0
+Text Label 3750 7000 1    50   ~ 0
 M1_1
 $Comp
 L power:Earth #PWR0109
 U 1 1 5FF3EB22
-P 3850 7000
-F 0 "#PWR0109" H 3850 6750 50  0001 C CNN
-F 1 "Earth" H 3850 6850 50  0001 C CNN
-F 2 "" H 3850 7000 50  0001 C CNN
-F 3 "~" H 3850 7000 50  0001 C CNN
-	1    3850 7000
+P 3650 7000
+F 0 "#PWR0109" H 3650 6750 50  0001 C CNN
+F 1 "Earth" H 3650 6850 50  0001 C CNN
+F 2 "" H 3650 7000 50  0001 C CNN
+F 3 "~" H 3650 7000 50  0001 C CNN
+	1    3650 7000
 	-1   0    0    1
 $EndComp
@@
 $EndComp
 $Comp
-L S6B-PH-SM4-TB_LF__SN_:S6B-PH-SM4-TB(LF)(SN) J1
-U 1 1 5FF58FC9
-P 4050 7300
-F 0 "J1" V 4450 7250 50  0000 L CNN
-F 1 "S6B-PH-SM4-TB(LF)(SN)" V 4350 6800 50  0000 L CNN
-F 2 "JST_S6B-PH-SM4-TB(LF)(SN)" H 4050 7300 50  0001 L BNN
-F 3 "" H 4050 7300 50  0001 L BNN
-F 4 "Manufacturer Recommendation" H 4050 7300 50  0001 L BNN "STANDARD"
-F 5 "JST" H 4050 7300 50  0001 L BNN "MANUFACTURER"
-	1    4050 7300
+L S8B-PH-SM4-TB_LF__SN_:S8B-PH-SM4-TB_LF__SN_ J1
+U 1 1 5FF1A68D
+P 4350 7000
+F 0 "J1" V 4754 7128 50  0000 L CNN
+F 1 "S8B-PH-SM4-TB_LF__SN_" V 4845 7128 50  0000 L CNN
+F 2 "S8BPHSM4TBLFSN" H 5100 7100 50  0001 L CNN
+F 3 "https://www.digikey.com/product-detail/en/jst-sales-america-inc/S8B-PH-SM4-TB-LF-SN/455-1755-1-ND/926852" H 5100 7000 50  0001 L CNN
+F 4 "Conn Shrouded Header (4 Sides) HDR 8 POS 2mm Solder RA Side Entry SMD T/R" H 5100 6900 50  0001 L CNN "Description"
+F 5 "5.5" H 5100 6800 50  0001 L CNN "Height"
+F 6 "JST (JAPAN SOLDERLESS TERMINALS)" H 5100 6700 50  0001 L CNN "Manufacturer_Name"
+F 7 "S8B-PH-SM4-TB(LF)(SN)" H 5100 6600 50  0001 L CNN "Manufacturer_Part_Number"
+F 8 "" H 5100 6500 50  0001 L CNN "Mouser Part Number"
+F 9 "" H 5100 6400 50  0001 L CNN "Mouser Price/Stock"
+F 10 "S8B-PH-SM4-TB(LF)(SN)" H 5100 6300 50  0001 L CNN "Arrow Part Number"
+F 11 "https://www.arrow.com/en/products/s8b-ph-sm4-tb-lf-sn/jst-manufacturing" H 5100 6200 50  0001 L CNN "Arrow Price/Stock"
+	1    4350 7000
 	0    1    1    0
 $EndComp
+NoConn ~ 4350 7900
+Text Label 3950 7000 1    50   ~ 0
+P0.21
+Text Label 4050 7000 1    50   ~ 0
+P1.00
 $EndSCHEMATC

Commit message: Type-C built-in power
Parts:
- removed H1, H2: MountingHole_Pad, symbol Mechanical:MountingHole_Pad
- added C19: 4.7uF 0603, Capacitors:0603, symbol pbrick-rescue:CAPACITOR_NP_0603-MF_Passives
- added C20, C21, C22, C23: 1uF 0603, Capacitors:0603, symbol pbrick-rescue:CAPACITOR_NP_0603-MF_Passives
- added C24: 100nF 0603, Capacitors:0603, symbol pbrick-rescue:CAPACITOR_NP_0603-MF_Passives
- added D1: ESDA25W, Common:SOT65P210X110-3N, symbol ESDA25W:ESDA25W
- added D2, D4: ESDA25P35-1U1M, TVS_ESDA25P35-1U1M, symbol ESDA25P35-1U1M:ESDA25P35-1U1M
- added D3: D_Schottky, Common:RESC0402X15N, symbol Device:D_Schottky
- added J2: UJC-HP-3-SMT-TR, CUI_UJC-HP-3-SMT-TR, symbol UJC-HP-3-SMT-TR:UJC-HP-3-SMT-TR
- added Q1, Q2: SSM6J507NU, TRANS_SSM6J507NU,LF, symbol SSM6J507NU_LF:SSM6J507NU,LF
- added R10: 22K Ω 0603, Resistors:0603, symbol pbrick-rescue:RESISTOR_0603-MF_Passives
- added R11: 100K Ω 0603, Resistors:0603, symbol pbrick-rescue:RESISTOR_0603-MF_Passives
- added R12: 100 Ω 0603, Resistors:0603, symbol pbrick-rescue:RESISTOR_0603-MF_Passives
- added R13, R8: 1K Ω 0603, Resistors:0603, symbol pbrick-rescue:RESISTOR_0603-MF_Passives
- added R7: 470 Ω 0603, Resistors:0603, symbol pbrick-rescue:RESISTOR_0603-MF_Passives
- added U4: STUSB4500QTR, QFN50P400X400X90-25N, symbol STUSB4500QTR:STUSB4500QTR
Connections:
- net labels added: DISCH, VBUS, VBUS_EN_SNK
- wire segments 97 -> 163
- no-connect marks 9 -> 17
Other:
- moved on the sheet: C1, C10, C11, C12, C13, C14, C15, C16, C3, C4, C6, C7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

Commit message: USB-PD Type-C Support
Parts:
- D3: footprint Common:RESC0402X15N -> Resistor_SMD:R_0603_1608Metric; Description DIODE SCHOTTKY 30V 100MA 0402 -> Diode Schottky 40V 200mA Surface Mount 0603 (1608 Metric); Digi-Key_PN 641-1675-1-ND -> CD0603-B0240RCT-ND; MPN CDBQR0130L-HF -> CD0603-B0240R; Manufacturer Comchip Technology -> Bourns Inc.
- U4: Description (none) -> USB-PD I2C Controller; Digi-Key_PN (none) -> 497-18060-1-ND; MANUFACTURER STMicroelectronics -> (none); MPN (none) -> STUSB4500QTR; Manufacturer (none) -> STMicroelectronics; PARTREV 2 -> (none); STANDARD IPC-7351B -> (none)
Connections:
- net VBUS: no longer C21.2, U4.24 (VDD)
- net at Q1.4, Q1.8, Q2.4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: now also C21.2, U4.24 (VDD)
