File: board/pbrick.sch (KiCad schematic (older format))
At the start: 53 parts, among them J1 S8B-PH-SM4-TB_LF__SN_, J2 UJC-HP-3-SMT-TR, J3 QWIIC, J5 U.FL2PIN, J6 TC2030-IDC-NL, Q1 SSM6J507NU, Q2 SSM6J507NU, U1 TB67H420FTG(O,EL), U2 MIC5219-3.3YML-TR, U3 ADP3330ARTZ-5-RL7, U4 STUSB4500QTR

Commit message: Added 3-axis sensor Added dedicate PWM driver Added 2 MOLEX connectors 3x5 (24mm x 40mm)
Parts:
- removed J1: S8B-PH-SM4-TB_LF__SN_, S8BPHSM4TBLFSN, symbol S8B-PH-SM4-TB_LF__SN_:S8B-PH-SM4-TB_LF__SN_
- added C20: 10nF 0402, Capacitors:0402, symbol pbrick-rescue:CAPACITOR_NP_0603-MF_Passives
- added C21, C26: 100nF 0402, Capacitors:0402, symbol pbrick-rescue:CAPACITOR_NP_0603-MF_Passives
- added M0, M1: 5055680471, MOLEX_5055680471, symbol 5055680471:5055680471
- added U6: 2533020201601, Package_LGA:LGA-12_2x2mm_P0.5mm, symbol pbrick:2533020201601
- added U7: PCA9624, Package_DFN_QFN:QFN-24-1EP_5x5mm_P0.65mm_EP3.2x3.2mm_ThermalVias, symbol pbrick:PCA9624
- C1, C6: value 470nF 0603 -> 470nF 0402; footprint Capacitors:0603 -> Capacitors:0402
- C10: renamed from C22; value 1uF 0603 -> 1uF 0402; footprint Capacitors:0603 -> Capacitors:0402
- C11: renamed from C9; value 22pF 0603 -> 22pF 0402; footprint Capacitors:0603 -> Capacitors:0402
- C12: renamed from C10; value 22pF 0603 -> 22pF 0402; footprint Capacitors:0603 -> Capacitors:0402
- C13: renamed from C11; value 22pF 0603 -> 22pF 0402; footprint Capacitors:0603 -> Capacitors:0402
- C14: renamed from C12; value 22pF 0603 -> 22pF 0402; footprint Capacitors:0603 -> Capacitors:0402
- C15: renamed from C13; value 22pF 0603 -> 22pF 0402; footprint Capacitors:0603 -> Capacitors:0402
- C17: renamed from C14; value 270pF 0603 -> 270pF 0402; footprint Capacitors:0603 -> Capacitors:0402
- C18: renamed from C15; value 100nF 0603 -> 100nF 0402; footprint Capacitors:0603 -> Capacitors:0402
- C2: renamed from C19; value 4.7uF 0603 -> 4.7uF 0402; footprint Capacitors:0603 -> Capacitors:0402
- C22: renamed from C8; value 1uF 0603 -> 1uF 0402; footprint Capacitors:0603 -> Capacitors:0402
- C23: renamed from C7; value 100nF 0603 -> 100nF 0402; footprint Capacitors:0603 -> Capacitors:0402
- C3, C4: footprint Capacitors:0603 -> Capacitors:0402
- C5: renamed from C20; value 1uF 0603 -> 1uF 0402; footprint Capacitors:0603 -> Capacitors:0402
- C7: renamed from C24; value 100nF 0603 -> 100nF 0402; footprint Capacitors:0603 -> Capacitors:0402
- C8: renamed from C21; value 1uF 0603 -> 1uF 0402; footprint Capacitors:0603 -> Capacitors:0402
- C9: renamed from C23; value 1uF 0603 -> 1uF 0402; footprint Capacitors:0603 -> Capacitors:0402
- D2: renamed from D1; footprint Common:SOT65P210X110-3N -> Package_TO_SOT_SMD:SOT-323_SC-70
- R1: renamed from R7; value 470 Ω 0603 -> 470 Ω 0402; footprint Resistors:0603 -> Resistors:0402
- R10: renamed from R3; value 140 Ω 0603 -> 140 Ω 0402; footprint Resistors:0603 -> Resistors:0402
- R11: renamed from R9; footprint Resistors:0603 -> Resistors:0402
- R12: renamed from R4; value 2.2K Ω 0603 -> 2.2K Ω 0402; footprint Resistors:0603 -> Resistors:0402
- R13: renamed from R5; value 2.2K Ω 0603 -> 2.2K Ω 0402; footprint Resistors:0603 -> Resistors:0402
- R2: renamed from R8; value 1K Ω 0603 -> 1K Ω 0402; footprint Resistors:0603 -> Resistors:0402
- R3: renamed from R10; value 22K Ω 0603 -> 22K Ω 0402; footprint Resistors:0603 -> Resistors:0402
- R4: renamed from R11; value 100K Ω 0603 -> 100K Ω 0402; footprint Resistors:0603 -> Resistors:0402
- R5: renamed from R12; value 100 Ω 0603 -> 100 Ω 0402; footprint Resistors:0603 -> Resistors:0402
- R6: renamed from R13; value 1K Ω 0603 -> 1K Ω 0402; footprint Resistors:0603 -> Resistors:0402
- R7: renamed from R6; value 10K 0603 -> 10K 0402; footprint Resistors:0603 -> Resistors:0402
- R8: renamed from R1; value 85 Ω 0603 -> 85 Ω 0402; footprint Resistors:0603 -> Resistors:0402
- R9: renamed from R2; value 85 Ω 0603 -> 85 Ω 0402; footprint Resistors:0603 -> Resistors:0402
- renumbered C16 to C19, D2 to D1, D6 to D4, D4 to D5, D5 to D6, J2 to J1, J6 to J2, J5 to J3, J3 to J4, U2 to U1, U3 to U2, U4 to U3, U1 to U5
Connections:
- net labels added: +2V8, +3.3VA, PCA9624_0, PCA9624_1, PCA9624_2, PCA9624_3, PCA9624_4, PCA9624_5, PCA9624_6, PCA9624_7
- net labels removed: VS, VSS
- wire segments 157 -> 199
- no-connect marks 16 -> 25
Other:
- note added: "Onboard Antenna: DNP C11 C12 C13, J3\n\nExternal Antenna: DNP C14, C15\n"
- note removed: "Onboard Antenna: DNP C6, C21 C26, J4\n\nExternal Antenna: DNP C27, C28\n"
- moved on the sheet: C10, C11, C12, C13, C14, C15, C17, C18, C19, C2, C22, C23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

Commit message: Updating footprints
Parts:
- C1, C6: value 470nF 0402 -> 470nF 0603; footprint Capacitors:0402 -> Capacitors:0603
- C10, C9: Description CAP CER 1UF 25V X7R 0603 -> CAP CER 1UF 10V X5R 0402; Digi-Key_PN 732-7994-1-ND -> 732-7489-1-ND; MPN 885012206076 -> 885012105012
- C11, C12, C13, C14, C15: Description CAP CER 22PF 16V C0G/NP0 0603 -> CAP CER 22PF 10V C0G/NP0 0402; Digi-Key_PN 732-7762-1-ND -> 732-7427-1-ND; MPN 885012006019 -> 885012005009
- C18, C26: Description CAP CER 0.1UF 25V X7R 0603 -> CAP CER 0.1UF 25V X5R 0402; Digi-Key_PN 732-7989-1-ND -> 732-7495-1-ND; MPN 885012206071 -> 885012105018
- C2: value 4.7uF 0402 -> 4.7uF 0603; footprint Capacitors:0402 -> Capacitors:0603
- C20: Description CAP CER 0.1UF 25V X7R 0603 -> CAP CER 0.1UF 25V X5R 0402
- C21: Digi-Key_PN 732-7989-1-ND -> 732-7495-1-ND; MPN 885012206071 -> 885012105018
- C22: Description CAP CER 1UF 16V X7R 0603 -> CAP CER 1UF 10V X5R 0402; Digi-Key_PN 732-7971-1-ND -> 732-7489-1-ND; MPN 885012206052 -> 885012105012
- C23: Description CAP CER 0.1UF 16V X7R 0603 -> CAP CER 0.1UF 25V X5R 0402; Digi-Key_PN 732-7965-1-ND -> 732-7495-1-ND; MPN 885012206046 -> 885012105018
- C5: value 1uF 0402 -> 1uF 0603; footprint Capacitors:0402 -> Capacitors:0603; Digi-Key_PN 732-7994-1-ND -> 732-7919-1-ND; MPN 885012206076 -> 885012106022
- C7: value 100nF 0402 -> 100nF 0603; footprint Capacitors:0402 -> Capacitors:0603
- C8: value 1uF 0402 -> 1uF 0603; footprint Capacitors:0402 -> Capacitors:0603; Description CAP CER 1UF 25V X7R 0603 -> CAP CER 1UF 25V X5R 0603; Digi-Key_PN 732-7994-1-ND -> 732-7919-1-ND; MPN 885012206076 -> 885012106022
- M0, M1: Description (none) -> CONN HEADER SMD 4POS 1.25MM; Digi-Key_PN (none) -> WM17035CT-ND; MANUFACTURER MOLEX -> (none); MPN (none) -> 5055680471; Manufacturer (none) -> Molex; PARTREV A -> (none); STANDARD Mnufacturer Recommendation -> (none)
- U7: footprint Package_DFN_QFN:QFN-24-1EP_5x5mm_P0.65mm_EP3.2x3.2mm_ThermalVias -> Package_DFN_QFN:QFN-24-1EP_5x5mm_P0.65mm_EP3.2x3.2mm

Commit message: Updating parts list
Parts:
- R1: Description RES SMD 470 OHM 5% 0.3W 0603 -> RES SMD 470 OHM 1% 1/5W 0402; Digi-Key_PN 511-1775-1-ND -> 541-10412-1-ND; MPN SDR03EZPJ471 -> RCS0402470RFKED; Manufacturer Rohm Semiconductor -> Vishay Dale
- R10: Description RES SMD 143 OHM 1% 1/4W 0603 -> RES SMD 150 OHM 1% 1/5W 0402; Digi-Key_PN 541-143SCT-ND -> 541-150YCT-ND; MPN CRCW0603143RFKEAHP -> CRCW0402150RFKEDHP
- R11: Description RES SMD 10K OHM 5% 1/4W 0603 -> RES SMD 5.1K OHM 5% 1/5W 0402; DigiKey_PN RHM10KDCT-ND -> 541-RCS04025K10JNEDCT-ND; MPN ESR03EZPJ103 -> RCS04025K10JNED; Manufacturer Rohm Semiconductor -> Vishay Dale
- R12, R13: Description RES SMD 2.2K OHM 5% 1/4W 0603 -> RES SMD 2.2K OHM 5% 1/5W 0402; Digi-Key_PN RHM2.2KDCT-ND -> 541-2914-1-ND; MPN ESR03EZPJ222 -> RCS04022K20JNED; Manufacturer Rohm Semiconductor -> Vishay Dale
- R2, R6: Description RES SMD 1K OHM 5% 1/4W 0603 -> RES SMD 1K OHM 5% 1/5W 0402; Digi-Key_PN RHM1.0KDCT-ND -> 541-2913-1-ND; MPN ESR03EZPJ102 -> RCS04021K00JNED; Manufacturer Rohm Semiconductor -> Vishay Dale
- R3: Description RES SMD 22K OHM 5% 1/4W 0603 -> RES SMD 22K OHM 5% 1/5W 0402; Digi-Key_PN RHM22KDCT-ND -> RHM1015CT-ND; MPN ESR03EZPJ223 -> ESR01MZPJ223
- R4: Description RES SMD 100K OHM 5% 1/4W 0603 -> RES SMD 100K OHM 5% 1/5W 0402; Digi-Key_PN RHM100KDCT-ND -> 541-2919-1-ND; MPN ESR03EZPJ104 -> RCS0402100KJNED; Manufacturer Rohm Semiconductor -> Vishay Dale
- R5: Description RES SMD 100 OHM 5% 1/4W 0603 -> RES SMD 100 OHM 1% 1/5W 0402; Digi-Key_PN RHM100DCT-ND -> 541-2886-1-ND; MPN ESR03EZPJ101 -> RCS0402100RFKED; Manufacturer Rohm Semiconductor -> Vishay Dale
- R7: Description RES SMD 10K OHM 5% 1/4W 0603 -> RES SMD 10K OHM 1% 1/5W 0402; Digi-Key_PN RHM10KDCT-ND -> 541-2894-1-ND; MPN ESR03EZPJ103 -> RCS040210K0FKED; Manufacturer Rohm Semiconductor -> Vishay Dale
- R8, R9: Description RES SMD 82 OHM 5% 1/4W 0603 -> RES SMD 82 OHM 1% 1/5W 0402; Digi-Key_PN RHM82DCT-ND -> 541-RCS040282R0FKEDCT-ND; MPN ESR03EZPJ820 -> RCS040282R0FKED; Manufacturer Rohm Semiconductor -> Vishay Dale

Commit message: Adding BOM information for PCA9632BS
Parts:
- C3: value 470pF -> 470pF 0402
- C4: value 2.2uF -> 2.2uF 0402
- U7: Description (none) -> IC LED DRIVER LINEAR DIM 24HVQFN; Digi-Key_PN (none) -> 568-5304-1-ND; MPN (none) -> PCA9624BS,118; Manufacturer (none) -> NXP USA Inc.
Changed lines of the file:
@@
 P 1800 2900
 F 0 "C4" H 1898 2942 45  0000 L CNN
-F 1 "2.2uF" H 1898 2858 45  0000 L CNN
+F 1 "2.2uF 0402" H 1898 2858 45  0000 L CNN
 F 2 "Capacitors:0402" H 2050 2810 20  0001 C CNN
 F 3 "https://katalog.we-online.de/pbs/datasheet/885012106018.pdf" H 1800 2900 60  0001 C CNN
@@
 P 1800 2500
 F 0 "C3" H 1898 2542 45  0000 L CNN
-F 1 "470pF" H 1898 2458 45  0000 L CNN
+F 1 "470pF 0402" H 1898 2458 45  0000 L CNN
 F 2 "Capacitors:0402" H 2050 2410 20  0001 C CNN
 F 3 "CAP CER 2.2UF 16V X5R 0603" H 1800 2500 60  0001 C CNN
@@
 F 2 "Package_DFN_QFN:QFN-24-1EP_5x5mm_P0.65mm_EP3.2x3.2mm" H 11450 1800 50  0001 C CNN
 F 3 "https://www.nxp.com/docs/en/data-sheet/PCA9624.pdf" H 11450 1800 50  0001 C CNN
+F 4 "NXP USA Inc." H 11400 1800 50  0001 C CNN "Manufacturer"
+F 5 "PCA9624BS,118" H 11400 1800 50  0001 C CNN "MPN"
+F 6 "568-5304-1-ND" H 11400 1800 50  0001 C CNN "Digi-Key_PN"
+F 7 "IC LED DRIVER LINEAR DIM 24HVQFN" H 11400 1800 50  0001 C CNN "Description"
 	1    11400 1800
 	1    0    0    -1

Commit message: Fixes design defect with 0402 resistor pads Adds NXP LED driver DigiKey Part information for ordering Adds more space for SWD connector Spaces out QWIIC and USB-C connector
Parts:
- C1, C2, C5, C6, C7, C8: footprint Capacitors:0603 -> Capacitor_SMD:C_0603_1608Metric
- C10, C11, C12, C13, C14, C15, C17, C18, C20, C21, C22, C23, C26, C3, C4, C9: footprint Capacitors:0402 -> Capacitor_SMD:C_0402_1005Metric
- R1, R10, R11, R12, R13, R2, R3, R4, R5, R6, R7, R8, R9: footprint Resistors:0402 -> Resistor_SMD:R_0402_1005Metric

Commit message: Correct schematic defect where Q2 was not routed on both ends
Connections:
- net VDD: now also C8.2, Q1.4, Q1.8, Q2.4, Q2.8, R4.1, U3.24 (VDD)
Changed lines of the file:
@@
 Text Label 12850 2550 2    50   ~ 0
 PCA9624_7
+Wire Wire Line
+	3400 4450 3400 4350
+Wire Wire Line
+	3400 4350 3800 4350
+Wire Wire Line
+	3800 4350 3800 4450
+Connection ~ 3400 4450
+Connection ~ 3800 4450
 $EndSCHEMATC
