File: board/pbrick.sch (KiCad schematic (older format))
At the start: 58 parts, among them J1 UJC-HP-3-SMT-TR, J2 TC2030-IDC-NL, J3 U.FL2PIN, J4 QWIIC, M0 5055680471, M1 5055680471, Q1 SSM6J507NU, Q2 SSM6J507NU, U1 MIC5219-3.3YML-TR, U2 ADP3330ARTZ-5-RL7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

Commit message: Updating layout
Parts:
- U7: footprint Package_DFN_QFN:QFN-24-1EP_5x5mm_P0.65mm_EP3.2x3.2mm -> Package_DFN_QFN:QFN-24-1EP_4x4mm_P0.5mm_EP2.65x2.65mm_ThermalVias
Connections:
- net labels removed: Earth
- wire segments 196 -> 203
Other:
- moved on the sheet: C10, C8, C9
Changed lines of the file:
@@
 U 1 1 5F248942
 P 11700 5250
-F 0 "C23" V 11600 4800 45  0000 L CNN
-F 1 "100nF 0402" V 11600 4900 45  0000 L CNN
+F 0 "C23" V 11550 4750 45  0000 L CNN
+F 1 "100nF 0402" V 11550 4900 45  0000 L CNN
 F 2 "Capacitor_SMD:C_0402_1005Metric" H 11950 5160 20  0001 C CNN
 F 3 "https://www.we-online.de/katalog/datasheet/885012106015.pdf" H 11700 5250 60  0001 C CNN
@@
 U 1 1 5F24CFB9
 P 11700 5000
-F 0 "C22" V 11850 4650 45  0000 L CNN
+F 0 "C22" V 11850 4600 45  0000 L CNN
 F 1 "1uF 0402" V 11850 4750 45  0000 L CNN
 F 2 "Capacitor_SMD:C_0402_1005Metric" H 11950 4910 20  0001 C CNN
@@
 	2750 6300 2650 6300
 Wire Wire Line
-	2650 6300 2650 6350
-Wire Wire Line
 	2650 6400 2750 6400
-$Comp
-L power:Earth #PWR014
-U 1 1 60249C39
-P 2650 6350
-F 0 "#PWR014" H 2650 6100 50  0001 C CNN
-F 1 "Earth" H 2650 6200 50  0001 C CNN
-F 2 "" H 2650 6350 50  0001 C CNN
-F 3 "~" H 2650 6350 50  0001 C CNN
-	1    2650 6350
-	0    1    1    0
-$EndComp
-Connection ~ 2650 6350
-Wire Wire Line
-	2650 6350 2650 6400
 NoConn ~ 2750 6700
 NoConn ~ 2750 5900
@@
 L pbrick-rescue:CAPACITOR_NP_0603-MF_Passives C8
 U 1 1 6027246D
-P 4700 5450
-F 0 "C8" V 4550 5400 45  0000 L CNN
-F 1 "1uF 0603" V 4550 5550 45  0000 L CNN
-F 2 "Capacitor_SMD:C_0603_1608Metric" H 4950 5360 20  0001 C CNN
-F 3 "https://www.we-online.de/katalog/datasheet/885012006019.pdf" H 4700 5450 60  0001 C CNN
-F 4 "732-7919-1-ND" H 4700 5450 50  0001 C CNN "Digi-Key_PN"
-F 5 "Würth Elektronik" H 4700 5450 50  0001 C CNN "Manufacturer"
-F 6 "885012106022" H 4700 5450 50  0001 C CNN "MPN"
-F 7 "CAP CER 1UF 25V X5R 0603" H 4700 5450 50  0001 C CNN "Description"
-	1    4700 5450
+P 4800 5450
+F 0 "C8" V 4800 5950 45  0000 L CNN
+F 1 "1uF 0603" V 4800 5600 45  0000 L CNN
+F 2 "Capacitor_SMD:C_0603_1608Metric" H 5050 5360 20  0001 C CNN
+F 3 "https://www.we-online.de/katalog/datasheet/885012006019.pdf" H 4800 5450 60  0001 C CNN
+F 4 "732-7919-1-ND" H 4800 5450 50  0001 C CNN "Digi-Key_PN"
+F 5 "Würth Elektronik" H 4800 5450 50  0001 C CNN "Manufacturer"
+F 6 "885012106022" H 4800 5450 50  0001 C CNN "MPN"
+F 7 "CAP CER 1UF 25V X5R 0603" H 4800 5450 50  0001 C CNN "Description"
+	1    4800 5450
 	0    1    1    0
 $EndComp
@@
 L pbrick-rescue:CAPACITOR_NP_0603-MF_Passives C9
 U 1 1 6028C5EF
-P 4700 6100
-F 0 "C9" H 4650 6400 45  0000 L CNN
-F 1 "1uF 0402" H 4300 6400 45  0000 L CNN
-F 2 "Capacitor_SMD:C_0402_1005Metric" H 4950 6010 20  0001 C CNN
-F 3 "https://www.we-online.de/katalog/datasheet/885012006019.pdf" H 4700 6100 60  0001 C CNN
-F 4 "732-7489-1-ND" H 4700 6100 50  0001 C CNN "Digi-Key_PN"
-F 5 "Würth Elektronik" H 4700 6100 50  0001 C CNN "Manufacturer"
-F 6 "885012105012" H 4700 6100 50  0001 C CNN "MPN"
-F 7 "CAP CER 1UF 10V X5R 0402" H 4700 6100 50  0001 C CNN "Description"
-	1    4700 6100
-	-1   0    0    1
+P 4800 6050
+F 0 "C9" V 4700 6550 45  0000 L CNN
+F 1 "1uF 0402" V 4700 6200 45  0000 L CNN
+F 2 "Capacitor_SMD:C_0402_1005Metric" H 5050 5960 20  0001 C CNN
+F 3 "https://www.we-online.de/katalog/datasheet/885012006019.pdf" H 4800 6050 60  0001 C CNN
+F 4 "732-7489-1-ND" H 4800 6050 50  0001 C CNN "Digi-Key_PN"
+F 5 "Würth Elektronik" H 4800 6050 50  0001 C CNN "Manufacturer"
+F 6 "885012105012" H 4800 6050 50  0001 C CNN "MPN"
+F 7 "CAP CER 1UF 10V X5R 0402" H 4800 6050 50  0001 C CNN "Description"
+	1    4800 6050
+	0    1    1    0
 $EndComp
 Wire Wire Line
@@
 Text Label 4550 7000 0    50   ~ 0
 VBUS_EN_SNK
-Text Label 3000 5250 0    50   ~ 0
+Text Label 3000 5300 0    50   ~ 0
 VBUS_EN_SNK
 $Comp
@@
 Wire Wire Line
 	3350 5100 4600 5100
-Wire Wire Line
-	4600 5100 4600 5450
 Connection ~ 3350 4450
 Wire Wire Line
@@
 L pbrick-rescue:CAPACITOR_NP_0603-MF_Passives C10
 U 1 1 6028C11A
-P 4950 5800
-F 0 "C10" V 5100 5650 45  0000 L CNN
-F 1 "1uF 0402" V 5100 5800 45  0000 L CNN
-F 2 "Capacitor_SMD:C_0402_1005Metric" H 5200 5710 20  0001 C CNN
-F 3 "https://www.we-online.de/katalog/datasheet/885012006019.pdf" H 4950 5800 60  0001 C CNN
-F 4 "732-7489-1-ND" H 4950 5800 50  0001 C CNN "Digi-Key_PN"
-F 5 "Würth Elektronik" H 4950 5800 50  0001 C CNN "Manufacturer"
-F 6 "885012105012" H 4950 5800 50  0001 C CNN "MPN"
-F 7 "CAP CER 1UF 10V X5R 0402" H 4950 5800 50  0001 C CNN "Description"
-	1    4950 5800
-	1    0    0    -1
-$EndComp
-Wire Wire Line
-	4700 6000 4550 6000
-Connection ~ 4600 5450
-Wire Wire Line
-	4600 5450 4600 5600
-Wire Wire Line
-	4550 5900 4950 5900
+P 4800 5850
+F 0 "C10" V 4700 6350 45  0000 L CNN
+F 1 "1uF 0402" V 4700 6000 45  0000 L CNN
+F 2 "Capacitor_SMD:C_0402_1005Metric" H 5050 5760 20  0001 C CNN
+F 3 "https://www.we-online.de/katalog/datasheet/885012006019.pdf" H 4800 5850 60  0001 C CNN
+F 4 "732-7489-1-ND" H 4800 5850 50  0001 C CNN "Digi-Key_PN"
+F 5 "Würth Elektronik" H 4800 5850 50  0001 C CNN "Manufacturer"
+F 6 "885012105012" H 4800 5850 50  0001 C CNN "MPN"
+F 7 "CAP CER 1UF 10V X5R 0402" H 4800 5850 50  0001 C CNN "Description"
+	1    4800 5850
+	0    1    1    0
+$EndComp
 $Comp
 L TC2030-IDC-NL:TC2030-IDC-NL J2
@@
 	1    3950 750
 	0    -1   -1   0
-$EndComp
-$Comp
-L power:GND #PWR026
-U 1 1 601D9D5C
-P 4800 5450
-F 0 "#PWR026" H 4800 5200 50  0001 C CNN
-F 1 "GND" V 4800 5350 50  0000 R CNN
-F 2 "" H 4800 5450 50  0001 C CNN
-F 3 "" H 4800 5450 50  0001 C CNN
-	1    4800 5450
-	0    -1   -1   0
-$EndComp
-$Comp
-L power:GND #PWR028
-U 1 1 601DA948
-P 4950 5700
-F 0 "#PWR028" H 4950 5450 50  0001 C CNN
-F 1 "GND" V 4850 5550 50  0000 C CNN
-F 2 "" H 4950 5700 50  0001 C CNN
-F 3 "" H 4950 5700 50  0001 C CNN
-	1    4950 5700
-	-1   0    0    1
 $EndComp
 $Comp
@@
 U 1 1 60933210
 P 8950 3500
-F 0 "C20" H 8750 3550 45  0000 L CNN
+F 0 "C20" H 8700 3550 45  0000 L CNN
 F 1 "10nF 0402" H 8450 3650 45  0000 L CNN
 F 2 "Capacitor_SMD:C_0402_1005Metric" H 9200 3410 20  0001 C CNN
@@
 L power:GND #PWR0102
 U 1 1 6038E92C
-P 4700 6200
-F 0 "#PWR0102" H 4700 5950 50  0001 C CNN
-F 1 "GND" H 4850 6150 50  0000 C CNN
-F 2 "" H 4700 6200 50  0001 C CNN
-F 3 "" H 4700 6200 50  0001 C CNN
-	1    4700 6200
+P 4900 6150
+F 0 "#PWR0102" H 4900 5900 50  0001 C CNN
+F 1 "GND" H 5050 6100 50  0000 C CNN
+F 2 "" H 4900 6150 50  0001 C CNN
+F 3 "" H 4900 6150 50  0001 C CNN
+	1    4900 6150
 	1    0    0    -1
 $EndComp
@@
 Wire Wire Line
 	4600 7750 4600 7800
-$Comp
-L power:GND #PWR0111
-U 1 1 60488417
-P 4550 5700
-F 0 "#PWR0111" H 4550 5450 50  0001 C CNN
-F 1 "GND" V 4550 5600 50  0000 R CNN
-F 2 "" H 4550 5700 50  0001 C CNN
-F 3 "" H 4550 5700 50  0001 C CNN
-	1    4550 5700
-	0    -1   -1   0
-$EndComp
 Text Label 12600 4050 0    50   ~ 0
 P0.22
@@
 F 0 "U7" H 11400 2000 50  0000 C CNN
 F 1 "PCA9624" H 11400 1850 50  0000 C CNN
-F 2 "Package_DFN_QFN:QFN-24-1EP_5x5mm_P0.65mm_EP3.2x3.2mm" H 11450 1800 50  0001 C CNN
+F 2 "Package_DFN_QFN:QFN-24-1EP_4x4mm_P0.5mm_EP2.65x2.65mm_ThermalVias" H 11450 1800 50  0001 C CNN
 F 3 "https://www.nxp.com/docs/en/data-sheet/PCA9624.pdf" H 11450 1800 50  0001 C CNN
 F 4 "NXP USA Inc." H 11400 1800 50  0001 C CNN "Manufacturer"
@@
 Text Label 11550 1050 1    50   ~ 0
 P1.00
+Wire Wire Line
+	2650 6300 2650 6350
+$Comp
+L power:GND #PWR?
+U 1 1 606B7FE9
+P 2650 6350
+F 0 "#PWR?" H 2650 6100 50  0001 C CNN
+F 1 "GND" H 2650 6200 50  0000 C CNN
+F 2 "" H 2650 6350 50  0001 C CNN
+F 3 "" H 2650 6350 50  0001 C CNN
+	1    2650 6350
+	0    1    1    0
+$EndComp
+Connection ~ 2650 6350
+Wire Wire Line
+	2650 6350 2650 6400
+Wire Wire Line
+	4550 5900 4700 5900
+Wire Wire Line
+	4700 5900 4700 5850
+Wire Wire Line
+	4550 6000 4700 6000
+Wire Wire Line
+	4700 6000 4700 6050
+Wire Wire Line
+	4900 5850 4900 6050
+Wire Wire Line
+	4900 6150 4900 6050
+Connection ~ 4900 6050
+Wire Wire Line
+	4900 5450 4900 5850
+Wire Wire Line
+	4600 5100 4600 5450
+Connection ~ 4900 5850
+Wire Wire Line
+	4700 5450 4600 5450
+Connection ~ 4600 5450
+Wire Wire Line
+	4600 5450 4600 5600
+Wire Wire Line
+	3000 5300 3000 5250
+$Comp
+L pbrick-rescue:3.3V-SparkFun-PowerSymbols #SUPPLY?
+U 1 1 6074472E
+P 4550 5700
+F 0 "#SUPPLY?" H 4600 5700 45  0001 L BNN
+F 1 "3.3V" V 4550 5828 45  0000 L CNN
+F 2 "XXX-00000" V 4508 5827 60  0001 L CNN
+F 3 "" H 4550 5700 60  0001 C CNN
+	1    4550 5700
+	0    1    1    0
+$EndComp
+$Comp
+L power:PWR_FLAG #FLG?
+U 1 1 60780EF2
+P 4600 4450
+F 0 "#FLG?" H 4600 4525 50  0001 C CNN
+F 1 "PWR_FLAG" V 4600 4800 50  0000 C CNN
+F 2 "" H 4600 4450 50  0001 C CNN
+F 3 "~" H 4600 4450 50  0001 C CNN
+	1    4600 4450
+	1    0    0    -1
+$EndComp
+Connection ~ 4600 4450
 $EndSCHEMATC

Commit message: Updating part list. Missing alt 12v connector
Parts:
- removed D1, D5: ESDA25P35-1U1M, TVS_ESDA25P35-1U1M, symbol ESDA25P35-1U1M:ESDA25P35-1U1M
- removed D2: ESDA25W, Package_TO_SOT_SMD:SOT-323_SC-70, symbol ESDA25W:ESDA25W
- added JP1: SolderJumper_2_Bridged, Jumper:SolderJumper-2_P1.3mm_Bridged_Pad1.0x1.5mm, symbol Jumper:SolderJumper_2_Bridged
- added U8: ESDA25W5, Package_TO_SOT_SMD:SOT-353_SC-70-5, symbol pbrick:ESDA25W5
- D3: footprint Resistor_SMD:R_0603_1608Metric -> Diode_SMD:D_0402_1005Metric; Description Diode Schottky 40V 200mA Surface Mount 0603 (1608 Metric) -> DIODE SCHOTTKY 30V 200MA 0402; Digi-Key_PN CD0603-B0240RCT-ND -> 641-2081-1-ND; MPN CD0603-B0240R -> CDBQR0230R-HF; Manufacturer Bourns Inc. -> Comchip Technology
- D4: Description DIODE SCHOTTKY 30V 100MA 0402 -> DIODE SCHOTTKY 30V 200MA 0402; Digi-Key_PN 641-1675-1-ND -> 641-2081-1-ND; MPN CDBQR0130L-HF -> CDBQR0230R-HF
Connections:
- net labels added: VSS
- wire segments 203 -> 197
Other:
- moved on the sheet: C2

Commit message: Adding extra vin, manual routing
Parts:
- added J5: 5055670271, Common:5055670271, symbol 5055670271:5055670271
- M0, M1: Alt_MPN (none) -> 5055670451 (gold)
Connections:
- net GND: now also J5.2
- net VDD: now also J5.1
- no-connect marks 17 -> 19
Changed lines of the file:
@@
 F 6 "5055680471" V 12300 6500 50  0001 C CNN "MPN"
 F 7 "CONN HEADER SMD 4POS 1.25MM" V 12300 6500 50  0001 C CNN "Description"
+F 8 "5055670451 (gold)" V 12300 6500 50  0001 C CNN "Alt_MPN"
 	1    12300 6500
 	0    -1   -1   0
@@
 F 6 "Molex" V 11450 6500 50  0001 C CNN "Manufacturer"
 F 7 "CONN HEADER SMD 4POS 1.25MM" V 11450 6500 50  0001 C CNN "Description"
+F 8 "5055670451 (gold)" V 11450 6500 50  0001 C CNN "Alt_MPN"
 	1    11450 6500
 	0    -1   -1   0
@@
 	1    0    0    -1
 $EndComp
+$Comp
+L 5055670271:5055670271 J5
+U 1 1 60674A7B
+P 13250 6200
+F 0 "J5" V 13439 6328 60  0000 L CNN
+F 1 "5055670271" V 13545 6328 60  0000 L CNN
+F 2 "Common:5055670271" H 13650 5940 60  0001 C CNN
+F 3 "https://www.molex.com/pdm_docs/ps/5055650000-000.pdf" V 13598 6328 60  0001 L CNN
+F 4 "WM17038CT-ND" V 13250 6200 50  0001 C CNN "Digi-Key_PN"
+F 5 "Molex" V 13250 6200 50  0001 C CNN "Manufacturer"
+F 6 "5055670271" V 13250 6200 50  0001 C CNN "MPN"
+F 7 "CONN HEADER SMD R/A 2POS 1.25MM" V 13250 6200 50  0001 C CNN "Description"
+	1    13250 6200
+	0    1    1    0
+$EndComp
+NoConn ~ 12950 6200
+NoConn ~ 13050 6200
+$Comp
+L power:GND #PWR0114
+U 1 1 6068C110
+P 13150 6200
+F 0 "#PWR0114" H 13150 5950 50  0001 C CNN
+F 1 "GND" V 13150 6000 50  0000 C CNN
+F 2 "" H 13150 6200 50  0001 C CNN
+F 3 "" H 13150 6200 50  0001 C CNN
+	1    13150 6200
+	-1   0    0    1
+$EndComp
+$Comp
+L power:VDD #PWR0116
+U 1 1 6068C641
+P 13250 6200
+F 0 "#PWR0116" H 13250 6050 50  0001 C CNN
+F 1 "VDD" V 13250 6400 50  0000 C CNN
+F 2 "" H 13250 6200 50  0001 C CNN
+F 3 "" H 13250 6200 50  0001 C CNN
+	1    13250 6200
+	1    0    0    -1
+$EndComp

Commit message: Updating Board, schematic, generated files
Connections:
- net VDD: no longer U8.1
- net VSS: now also U8.1
Other:
- moved on the sheet: JP1
Changed lines of the file:
@@
 U 1 1 606451CC
 P 1750 6400
-F 0 "U8" H 1800 7000 50  0000 R CNN
-F 1 "ESDA25W5" H 1950 6900 50  0000 R CNN
+F 0 "U8" V 2000 7100 50  0000 R CNN
+F 1 "ESDA25W5" V 2000 6950 50  0000 R CNN
 F 2 "Package_TO_SOT_SMD:SOT-353_SC-70-5" H 1750 6400 50  0001 C CNN
 F 3 "https://www.mouser.com/datasheet/2/389/cd00064033-1796223.pdf" H 1750 6400 50  0001 C CNN
@@
 Wire Wire Line
 	1400 4950 1700 4950
-$Comp
-L power:VDD #PWR0104
-U 1 1 606BF5CF
-P 1600 6600
-F 0 "#PWR0104" H 1600 6450 50  0001 C CNN
-F 1 "VDD" H 1615 6773 50  0000 C CNN
-F 2 "" H 1600 6600 50  0001 C CNN
-F 3 "" H 1600 6600 50  0001 C CNN
-	1    1600 6600
-	-1   0    0    1
-$EndComp
 Wire Wire Line
 	1700 4950 1850 4950
@@
 L power:VDD #PWR0111
 U 1 1 6077858F
-P 5450 4250
-F 0 "#PWR0111" H 5450 4100 50  0001 C CNN
-F 1 "VDD" H 5465 4423 50  0000 C CNN
-F 2 "" H 5450 4250 50  0001 C CNN
-F 3 "" H 5450 4250 50  0001 C CNN
-	1    5450 4250
-	0    1    1    0
+P 5350 3850
+F 0 "#PWR0111" H 5350 3700 50  0001 C CNN
+F 1 "VDD" H 5365 4023 50  0000 C CNN
+F 2 "" H 5350 3850 50  0001 C CNN
+F 3 "" H 5350 3850 50  0001 C CNN
+	1    5350 3850
+	1    0    0    -1
 $EndComp
 $Comp
@@
 L power:VSS #PWR0113
 U 1 1 60793775
-P 5150 4250
-F 0 "#PWR0113" H 5150 4100 50  0001 C CNN
-F 1 "VSS" V 5168 4378 50  0000 L CNN
-F 2 "" H 5150 4250 50  0001 C CNN
-F 3 "" H 5150 4250 50  0001 C CNN
-	1    5150 4250
-	0    -1   -1   0
+P 5350 4150
+F 0 "#PWR0113" H 5350 4000 50  0001 C CNN
+F 1 "VSS" V 5368 4278 50  0000 L CNN
+F 2 "" H 5350 4150 50  0001 C CNN
+F 3 "" H 5350 4150 50  0001 C CNN
+	1    5350 4150
+	-1   0    0    1
 $EndComp
 Connection ~ 4600 4450
@@
 L Jumper:SolderJumper_2_Bridged JP1
 U 1 1 607BE31E
-P 5300 4250
-F 0 "JP1" H 5300 4455 50  0000 C CNN
-F 1 "SolderJumper_2_Bridged" H 5300 4364 50  0000 C CNN
-F 2 "Jumper:SolderJumper-2_P1.3mm_Bridged_Pad1.0x1.5mm" H 5300 4250 50  0001 C CNN
-F 3 "~" H 5300 4250 50  0001 C CNN
-	1    5300 4250
-	1    0    0    -1
+P 5350 4000
+F 0 "JP1" H 5350 4205 50  0000 C CNN
+F 1 "SolderJumper_2_Bridged" H 5350 4114 50  0000 C CNN
+F 2 "Jumper:SolderJumper-2_P1.3mm_Bridged_Pad1.0x1.5mm" H 5350 4000 50  0001 C CNN
+F 3 "~" H 5350 4000 50  0001 C CNN
+	1    5350 4000
+	0    -1   -1   0
 $EndComp
 $Comp
@@
 U 1 1 60674A7B
 P 13250 6200
-F 0 "J5" V 13439 6328 60  0000 L CNN
-F 1 "5055670271" V 13545 6328 60  0000 L CNN
+F 0 "J5" V 13400 6300 60  0000 L CNN
+F 1 "5055670271" V 13545 6328 60  0001 L CNN
 F 2 "Common:5055670271" H 13650 5940 60  0001 C CNN
 F 3 "https://www.molex.com/pdm_docs/ps/5055650000-000.pdf" V 13598 6328 60  0001 L CNN
@@
 	1    0    0    -1
 $EndComp
+$Comp
+L power:VSS #PWR?
+U 1 1 6067CFEC
+P 1600 6600
+F 0 "#PWR?" H 1600 6450 50  0001 C CNN
+F 1 "VSS" V 1617 6728 50  0000 L CNN
+F 2 "" H 1600 6600 50  0001 C CNN
+F 3 "" H 1600 6600 50  0001 C CNN
+	1    1600 6600
+	-1   0    0    1
+$EndComp
 $EndSCHEMATC
